File: pcb/tuner.kicad_pcb (KiCad board)
At the start: 2 copper layers, 0 parts

Commit message: Mostly finished layout.
Parts:
- added BT1: BATTERY, BATTERY, B.Cu at (130.0, 66.5)
- added C1: 10 uF, SM0805, F.Cu at (153.9, 69.2)
- added C10: 27 pF, SM0805, F.Cu at (119.0, 67.7)
- added C2: 100 nF, SM0805, F.Cu at (102.5, 76.3)
- added C3: 22 pF, SM0805, F.Cu at (148.0, 64.7)
- added C4: 10 uF, SM0805, F.Cu at (149.3, 71.4)
- added C5: 100 nF, SM0805, F.Cu at (105.0, 72.0)
- added C6: 100 nF, SM0805, F.Cu at (106.4, 60.2)
- added C7: 100 nF, SM0805, F.Cu at (104.1, 60.1)
- added C8: 100 nF, SM0805, F.Cu at (116.7, 70.8)
- added C9: 25 pF, SM0805, F.Cu at (119.0, 64.5)
- added D1: LED, SM0805, F.Cu at (79.2, 58.3)
- added D2: LED, SM0805, F.Cu at (79.2, 61.7)
- added L1: 2.2 uH, SM1008, F.Cu at (148.1, 68.5)
- added P1: PDI, pin_array_3x2, F.Cu at (111.3, 75.4)
- added R1: 420 K, SM0805, F.Cu at (148.1, 62.7)
- added R10: 27 Ohms, SM0805, F.Cu at (127.8, 69.8)
- added R11: 27 Ohms, SM0805, F.Cu at (127.8, 62.6)
- added R12: 10 K, SM0805, F.Cu at (109.8, 58.0)
- added R13: 27 Ohms, SM0805, F.Cu at (127.8, 66.2)
- added R14: 27 Ohms, SM0805, F.Cu at (140.2, 74.1)
- added R15: 18 Ohms, SM0805, F.Cu at (83.5, 58.3)
- added R16: 18 Ohms, SM0805, F.Cu at (83.5, 61.7)
- added R2: 180 K, SM0805, F.Cu at (151.6, 62.7)
- added R3: 10 K, SM0805, F.Cu at (104.9, 76.3)
- added R4: 10 K, SM0805, F.Cu at (116.7, 75.4)
- added R5: 10 K, SM0805, F.Cu at (103.9, 67.9)
- added R6: 27 Ohms, SM0805, F.Cu at (127.8, 59.0)
- added R7: 27 Ohms, SM0805, F.Cu at (140.2, 58.7)
- added R8: 27 Ohms, SM0805, F.Cu at (137.8, 74.1)
- added R9: 27 Ohms, SM0805, F.Cu at (127.8, 73.4)
- added SW1: SPST, DIP1, F.Cu at (158.0, 66.2)
- added SW2: <, SWITCH_YAY, F.Cu at (96.0, 73.0)
- added SW3: >, SWITCH_YAY, F.Cu at (96.0, 66.0)
- added SW4: Mode, SWITCH_YAY, F.Cu at (96.0, 57.0)
- added U1: TPS62240, SOT23-5-2, F.Cu at (152.0, 65.9)
- added U2: NKR131SB, LED_DISPLAY, F.Cu at (136.2, 66.4)
- added U3: ATXMEGA8E5, TQFP32-2, F.Cu at (111.2, 65.8)
- added Y1: 8 MHz, CRYSTAL_SMD, F.Cu at (123.4, 66.0)
Routing:
- net GND: track 0.00 -> 13.0 mm, vias 0 -> 2
- net N-0000029: track 0.00 -> 10.2 mm
- net N-0000031: track 0.00 -> 10.1 mm
- net N-0000046: track 0.00 -> 8.96 mm
- net N-0000027: track 0.00 -> 5.62 mm
- net VDD: track 0.00 -> 5.33 mm
- added copper zone on F.Cu, net GND
- added copper zone on F.Cu, net N-0000028
- added copper zone on F.Cu, net VDD
Other:
- board outline added: 89 x 24.5 mm
- net class Chip Power added: clearance 0.254, trace_width 0.508, via_dia 0.889, via_drill 0.635
- net class Supply Power added: clearance 0.254, trace_width 0.762, via_dia 0.889, via_drill 0.635
- board text added: "BT1"
- board text added: "Off"
- board text added: "On"
- board text added: "© 2014 Neil MacMillan Strobe Guitar Tuner r2 http://nrqm.ca/guitar-tuner"
