File: pcb/tuner.sch (KiCad schematic (older format))
At the start: 30 parts, among them P1 PDI, SW1 SPST, SW2 <, SW3 >, SW4 Mode, U1 TPS622312, U2 NKR131SB, U3 ATXMEGA8E5, X1 8 MHz

Commit message: Mostly finished layout.
Parts:
- removed C1: 2.2 uF, ~, symbol C
- removed U1: TPS622312, symbol TPS622312
- added C2, C5, C7: 100 nF, ~, symbol C
- added C3: 22 pF, ~, symbol C
- added C4: 10 uF, ~, symbol C
- added R1: 422 K, ~, symbol R
- added R12, R3, R5: 10 K, ~, symbol R
- added R2: 180 K, ~, symbol R
- added U1: TPS62240, ~, symbol TPS62240
- BT1: value BATT -> BATTERY; URL (none) -> http://www.digikey.ca/product-detail/en/BH2AAAPC/BH2AAA-PC-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
- C1: renamed from C2; value 4.7 uF -> 10 uF; URL (none) -> http://www.digikey.ca/product-detail/en/CC0805KKX5R5BB106/3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
- C10: renamed from C6; URL (none) -> http://www.digikey.ca/product-detail/en/C0805C270J5GACTU/39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
- C6: renamed from C3; URL (none) -> http://www.digikey.ca/product-detail/en/CC0805KKX5R5BB106/3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
- C8: renamed from C4; URL (none) -> http://www.digikey.ca/product-detail/en/CC0805KKX5R5BB106/3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
- C9: renamed from C5; URL (none) -> http://www.digikey.ca/product-detail/en/CL21C250JBANNNC/127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
- L1: URL http://www.digikey.ca/product-detail/en/LQM21PN2R2MC0D/490-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 -> http://www.digikey.ca/product-detail/en/LQM2HPN2R2MJ0L/490-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
- R10: renamed from R6; URL (none) -> http://www.digikey.ca/product-detail/en/ERJ-6ENF27R0V/P27.0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
- R11: renamed from R7; URL (none) -> http://www.digikey.ca/product-detail/en/ERJ-6ENF27R0V/P27.0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
- R13: renamed from R8; URL (none) -> http://www.digikey.ca/product-detail/en/ERJ-6ENF27R0V/P27.0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
- R14: renamed from R9; URL (none) -> http://www.digikey.ca/product-detail/en/ERJ-6ENF27R0V/P27.0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
- R15: renamed from R10; URL (none) -> http://www.digikey.ca/product-detail/en/RC0805FR-0718RL/311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
- R16: renamed from R11; URL (none) -> http://www.digikey.ca/product-detail/en/RC0805FR-0718RL/311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
- R4: renamed from R1; URL (none) -> http://www.digikey.ca/product-detail/en/RC0805FR-0710KL/311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
- R6: renamed from R2; URL (none) -> http://www.digikey.ca/product-detail/en/ERJ-6ENF27R0V/P27.0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
- R7: renamed from R3; URL (none) -> http://www.digikey.ca/product-detail/en/ERJ-6ENF27R0V/P27.0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
- R8: renamed from R4; URL (none) -> http://www.digikey.ca/product-detail/en/ERJ-6ENF27R0V/P27.0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
- R9: renamed from R5; URL (none) -> http://www.digikey.ca/product-detail/en/ERJ-6ENF27R0V/P27.0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
- SW2, SW3, SW4: URL (none) -> http://www.digikey.ca/product-detail/en/MJTP1243/679-2452-N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
- renumbered X1 to Y1
Connections:
- net GND: now also C2.1, C4.1, C5.1, C7.1, R2.1, U1.2 (GND)
- net VDD: now also L1.2, C3.2, C4.2, R1.2, R12.2, R3.1, R5.2; no longer C1.1, L1.1
- net at SW1.2: now also C1.1, U1.1 (VIN), U1.3 (EN)
- net at SW2.2, U3.5 (PA1): now also C2.2, R3.2
- net at SW3.2, U3.6 (PA0): now also C5.2, R5.1
- net at SW4.2, U3.28 (PD0): now also C7.2, R12.1
- new net: L1.1, U1.5 (SW)
- new net: C3.1, R1.1, R2.2, U1.4 (FB)
Other:
- moved on the sheet: C1, C10, C6, C8, C9, D1, D2, L1, P1, R10, R11, R13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
